Commit message: further sim app updates

File: deeprotor-simapp/bundle/opt/install/deeprotor_simulation_environment/share/deepracer_simulation_environment/urdf/macros.xacro (robot description, xacro)
@@ -1,112 +1,3 @@
 <?xml version="1.0"?>
-<robot name="racecar" xmlns:xacro="http://www.ros.org/wiki/xacro">
-<!-- inertial parameter macros -->
-<xacro:macro name="chassis_inertial_params">
-  <origin xyz="0.1477 0 0" rpy="0 0 0" />
-  <mass value="5.0" />
-  <inertia ixx="0.010609" ixy="0"          ixz="0"
-                          iyy="0.050409"   iyz="0"
-                                           izz="0.05865" />
-</xacro:macro>
-<xacro:macro name="left_wheels_inertial_params">
-  <origin xyz="0 0 -0.0125" rpy="0 0 0" />
-  <mass value="0.34055" />
-  <inertia ixx="0.00026046" ixy="0"          ixz="0"
-                            iyy="0.00026046" iyz="0"
-                                             izz="0.00041226" />
-</xacro:macro>
-<xacro:macro name="right_wheels_inertial_params">
-  <origin xyz="0 0 0.0125" rpy="0 0 0" />
-  <mass value="0.34055" />
-  <inertia ixx="0.00026046" ixy="0"          ixz="0"
-                            iyy="0.00026046" iyz="0"
-                                             izz="0.00041226" />
-</xacro:macro>
-<xacro:macro name="steering_hinge_inertial_params">
-  <origin xyz="0 0 0" rpy="0 0 0" />
-  <mass value="0.100" />
-  <inertia ixx="4E-06" ixy="0"           ixz="0"
-                            iyy="4E-06"  iyz="0"
-                                              izz="4E-06" />
-</xacro:macro>
-<!-- geometry macros -->
-<xacro:macro name="chassis_geometry">
-  <origin xyz="0 0 0" rpy="0 0 0" />
-  <geometry>
-      <mesh scale="0.6 0.6 0.6" filename="package://deepracer_simulation_environment/meshes/chassis.STL"/>
-  </geometry>
-</xacro:macro>
-<xacro:macro name="left_rear_wheel_geometry">
-  <origin xyz="0 0 0" rpy="0 0 0" />
-  <geometry>
-    <mesh scale="0.6 0.6 0.6" filename="package://deepracer_simulation_environment/meshes/left_rear_wheel.STL" />
-  </geometry>
-</xacro:macro>
-<xacro:macro name="right_rear_wheel_geometry">
-  <origin xyz="0 0 0" rpy="0 0 0" />
-  <geometry>
-    <mesh scale="0.6 0.6 0.6" filename="package://deepracer_simulation_environment/meshes/right_rear_wheel.STL" />
-  </geometry>
-</xacro:macro>
-<xacro:macro name="left_front_wheel_geometry">
-  <origin xyz="0 0 0" rpy="0 0 0" />
-  <geometry>
-    <mesh scale="0.6 0.6 0.6" filename="package://deepracer_simulation_environment/meshes/left_front_wheel.STL" />
-  </geometry>
-</xacro:macro>
-<xacro:macro name="right_front_wheel_geometry">
-  <origin xyz="0 0 0" rpy="0 0 0" />
-  <geometry>
-    <mesh scale="0.6 0.6 0.6" filename="package://deepracer_simulation_environment/meshes/right_front_wheel.STL" />
-  </geometry>
-</xacro:macro>
-<xacro:macro name="left_steering_hinge_geometry">
-  <origin xyz="0 0 0" rpy="0 0 0" />
-  <geometry>
-    <mesh scale="0.6 0.6 0.6" filename="package://deepracer_simulation_environment/meshes/left_steering_hinge.STL" />
-  </geometry>
-</xacro:macro>
-<xacro:macro name="right_steering_hinge_geometry">
-  <origin xyz="0 0 0" rpy="0 0 0" />
-  <geometry>
-    <mesh scale="0.6 0.6 0.6" filename="package://deepracer_simulation_environment/meshes/right_steering_hinge.STL" />
-  </geometry>
-</xacro:macro>
-<xacro:macro name="left_wheels_collision_geometry">
-  <origin xyz="0 0 -0.0125" rpy="0 0 0" />
-  <geometry>
-    <cylinder length="0.025" radius="0.03" />
-  </geometry>
-</xacro:macro>
-<xacro:macro name="right_wheels_collision_geometry">
-  <origin xyz="0 0 0.0125" rpy="0 0 0" />
-  <geometry>
-    <cylinder length="0.025" radius="0.03" />
-  </geometry>
-</xacro:macro>
-<!-- transmission macros -->
-<xacro:macro name="wheel_transmission" params="name">
-  <transmission name="${name}_transmission" type="SimpleTransmission">
-    <type>transmission_interface/SimpleTransmission</type>
-    <joint name="${name}_joint">
-      <hardwareInterface>EffortJointInterface</hardwareInterface>
-    </joint>
-    <actuator name="${name}_motor">
-      <hardwareInterface>EffortJointInterface</hardwareInterface>
-      <mechanicalReduction>1</mechanicalReduction>
-    </actuator>
-  </transmission>
-</xacro:macro>
-<xacro:macro name="steering_hinge_transmission" params="name">
-  <transmission name="${name}_transmission" type="SimpleTransmission">
-    <type>transmission_interface/SimpleTransmission</type>
-    <joint name="${name}_joint">
-      <hardwareInterface>EffortJointInterface</hardwareInterface>
-    </joint>
-    <actuator name="${name}_motor">
-      <hardwareInterface>EffortJointInterface</hardwareInterface>
-      <mechanicalReduction>1</mechanicalReduction>
-    </actuator>
-  </transmission>
-</xacro:macro>
+<robot name="drone" xmlns:xacro="http://www.ros.org/wiki/xacro">
 </robot>

File: deeprotor-simapp/bundle/opt/install/deeprotor_simulation_environment/share/deepracer_simulation_environment/urdf/materials.xacro (robot description, xacro)
@@ -1,4 +1,4 @@
 <?xml version="1.0"?>
-<robot name="racecar" xmlns:xacro="http://www.ros.org/wiki/xacro">
+<robot name="drone" xmlns:xacro="http://www.ros.org/wiki/xacro">
 <material name="black">
   <color rgba="0.0 0.0 0.0 1.0"/>
