Commit message: added rotors files and adjusted launch config

File: deeprotor-simapp/bundle/opt/install/deeprotor_simulation_environment/share/deepracer_simulation_environment/urdf/drone.xacro (robot description, xacro)
@@ -1,5 +1,4 @@
 <?xml version="1.0"?>
 <robot name="drone" xmlns:xacro="http://www.ros.org/wiki/xacro">
-  <xacro:include filename="$(find deeprotor_simulation_environment)/urdf/macros.xacro" />
   <!-- zed camera -->
   <link name="zed_camera_link">
@@ -24,6 +23,5 @@
   </link>
   <joint name="zed_camera_joint" type="fixed">
-    <origin xyz="0.20 0 0.134" rpy="0 0.261799 0"/>
-    <parent link="chassis"/>
+    <origin xyz="0.0 0.0 -0.08" rpy="0.0 0.1 2.3" />
     <child link="zed_camera_link"/>
     <axis xyz="0 0 1" />
