Commit message: add base link parent

File: deeprotor_ws/src/deeprotor_simulation_environment/urdf/drone.xacro (robot description, xacro)
@@ -1,4 +1,5 @@
 <?xml version="1.0"?>
 <robot name="drone" xmlns:xacro="http://www.ros.org/wiki/xacro">
+  <link name="base_link" />
   <!-- zed camera -->
   <link name="zed_camera_link">
@@ -24,4 +25,5 @@
   <joint name="zed_camera_joint" type="fixed">
     <origin xyz="0.0 0.0 -0.08" rpy="0.0 0.1 2.3" />
+    <parent link="base_link"/>
     <child link="zed_camera_link"/>
     <axis xyz="0 0 1" />

Commit message: use drone/base_link

File: deeprotor_ws/src/deeprotor_simulation_environment/urdf/drone.xacro (robot description, xacro)
@@ -1,5 +1,4 @@
 <?xml version="1.0"?>
 <robot name="drone" xmlns:xacro="http://www.ros.org/wiki/xacro">
-  <link name="base_link" />
   <!-- zed camera -->
   <link name="zed_camera_link">
@@ -25,5 +24,5 @@
   <joint name="zed_camera_joint" type="fixed">
     <origin xyz="0.0 0.0 -0.08" rpy="0.0 0.1 2.3" />
-    <parent link="base_link"/>
+    <parent link="drone/base_link"/>
     <child link="zed_camera_link"/>
     <axis xyz="0 0 1" />

Commit message: shrink camera size

File: deeprotor_ws/src/deeprotor_simulation_environment/urdf/drone.xacro (robot description, xacro)
@@ -11,5 +11,5 @@
       <origin xyz="0 0 0" rpy="0 0 0"/>
       <geometry>
-        <box size="0.033 0.175 0.030"/>
+        <box size="0.01 0.05 0.015"/>
       </geometry>
     </collision>
@@ -17,5 +17,5 @@
       <origin xyz="0 0 0" rpy="0 0 0"/>
       <geometry>
-        <box size="0.033 0.175 0.030"/>
+        <box size="0.01 0.05 0.015"/>
       </geometry>
       <material name="red"/>

Commit message: move camera up to prevent tipping over

File: deeprotor_ws/src/deeprotor_simulation_environment/urdf/drone.xacro (robot description, xacro)
@@ -5,9 +5,9 @@
     <inertial>
       <mass value="1e-3" />
-      <origin xyz="0 0 0" rpy="0 0 0"/>
+      <origin xyz="0 0.02 0" rpy="0 0 0"/>
       <inertia ixx="1e-6" ixy="0" ixz="0" iyy="1e-6" iyz="0" izz="1e-6" />
     </inertial>
     <collision>
-      <origin xyz="0 0 0" rpy="0 0 0"/>
+      <origin xyz="0 0.02 0" rpy="0 0 0"/>
       <geometry>
         <box size="0.01 0.05 0.015"/>
@@ -15,5 +15,5 @@
     </collision>
     <visual>
-      <origin xyz="0 0 0" rpy="0 0 0"/>
+      <origin xyz="0 0.02 0" rpy="0 0 0"/>
       <geometry>
         <box size="0.01 0.05 0.015"/>
@@ -23,5 +23,5 @@
   </link>
   <joint name="zed_camera_joint" type="fixed">
-    <origin xyz="0.0 0.0 -0.08" rpy="0.0 0.1 2.3" />
+    <origin xyz="0.0 0.02 -0.08" rpy="0.0 0.1 2.3" />
     <parent link="drone/base_link"/>
     <child link="zed_camera_link"/>
@@ -34,10 +34,10 @@
     <inertial>
       <mass value="1e-3" />
-      <origin xyz="0 0 0" rpy="0 0 0"/>
+      <origin xyz="0 0.02 0" rpy="0 0 0"/>
       <inertia ixx="1e-6" ixy="0" ixz="0" iyy="1e-6" iyz="0" izz="1e-6" />
     </inertial>
   </link>
   <joint name="zed_camera_left_joint" type="fixed">
-    <origin xyz="0 0 0" rpy="0 0 0"/>
+    <origin xyz="0 0.02 0" rpy="0 0 0"/>
     <parent link="zed_camera_link"/>
     <child link="camera_link"/>

Commit message: move camera up

File: deeprotor_ws/src/deeprotor_simulation_environment/urdf/drone.xacro (robot description, xacro)
@@ -5,9 +5,9 @@
     <inertial>
       <mass value="1e-3" />
-      <origin xyz="0 0.02 0" rpy="0 0 0"/>
+      <origin xyz="0 0 0.05" rpy="0 0 0"/>
       <inertia ixx="1e-6" ixy="0" ixz="0" iyy="1e-6" iyz="0" izz="1e-6" />
     </inertial>
     <collision>
-      <origin xyz="0 0.02 0" rpy="0 0 0"/>
+      <origin xyz="0 0 0.05" rpy="0 0 0"/>
       <geometry>
         <box size="0.01 0.05 0.015"/>
@@ -15,5 +15,5 @@
     </collision>
     <visual>
-      <origin xyz="0 0.02 0" rpy="0 0 0"/>
+      <origin xyz="0 0 0.05" rpy="0 0 0"/>
       <geometry>
         <box size="0.01 0.05 0.015"/>
@@ -23,5 +23,5 @@
   </link>
   <joint name="zed_camera_joint" type="fixed">
-    <origin xyz="0.0 0.02 -0.08" rpy="0.0 0.1 2.3" />
+    <origin xyz="0.0 0.0 0.05" rpy="0.0 0.1 2.3" />
     <parent link="drone/base_link"/>
     <child link="zed_camera_link"/>
@@ -34,10 +34,10 @@
     <inertial>
       <mass value="1e-3" />
-      <origin xyz="0 0.02 0" rpy="0 0 0"/>
+      <origin xyz="0 0 0.05" rpy="0 0 0"/>
       <inertia ixx="1e-6" ixy="0" ixz="0" iyy="1e-6" iyz="0" izz="1e-6" />
     </inertial>
   </link>
   <joint name="zed_camera_left_joint" type="fixed">
-    <origin xyz="0 0.02 0" rpy="0 0 0"/>
+    <origin xyz="0 0 0.05" rpy="0 0 0"/>
     <parent link="zed_camera_link"/>
     <child link="camera_link"/>

Commit message: reduce camera adustment

File: deeprotor_ws/src/deeprotor_simulation_environment/urdf/drone.xacro (robot description, xacro)
@@ -5,9 +5,9 @@
     <inertial>
       <mass value="1e-3" />
-      <origin xyz="0 0 0.05" rpy="0 0 0"/>
+      <origin xyz="0 0 0.005" rpy="0 0 0"/>
       <inertia ixx="1e-6" ixy="0" ixz="0" iyy="1e-6" iyz="0" izz="1e-6" />
     </inertial>
     <collision>
-      <origin xyz="0 0 0.05" rpy="0 0 0"/>
+      <origin xyz="0 0 0.005" rpy="0 0 0"/>
       <geometry>
         <box size="0.01 0.05 0.015"/>
@@ -15,5 +15,5 @@
     </collision>
     <visual>
-      <origin xyz="0 0 0.05" rpy="0 0 0"/>
+      <origin xyz="0 0 0.005" rpy="0 0 0"/>
       <geometry>
         <box size="0.01 0.05 0.015"/>
@@ -23,5 +23,5 @@
   </link>
   <joint name="zed_camera_joint" type="fixed">
-    <origin xyz="0.0 0.0 0.05" rpy="0.0 0.1 2.3" />
+    <origin xyz="0.0 0.0 0.005" rpy="0.0 0.1 2.3" />
     <parent link="drone/base_link"/>
     <child link="zed_camera_link"/>
@@ -34,10 +34,10 @@
     <inertial>
       <mass value="1e-3" />
-      <origin xyz="0 0 0.05" rpy="0 0 0"/>
+      <origin xyz="0 0 0.005" rpy="0 0 0"/>
       <inertia ixx="1e-6" ixy="0" ixz="0" iyy="1e-6" iyz="0" izz="1e-6" />
     </inertial>
   </link>
   <joint name="zed_camera_left_joint" type="fixed">
-    <origin xyz="0 0 0.05" rpy="0 0 0"/>
+    <origin xyz="0 0 0.005" rpy="0 0 0"/>
     <parent link="zed_camera_link"/>
     <child link="camera_link"/>

Commit message: adjust camera z again

File: deeprotor_ws/src/deeprotor_simulation_environment/urdf/drone.xacro (robot description, xacro)
@@ -5,9 +5,9 @@
     <inertial>
       <mass value="1e-3" />
-      <origin xyz="0 0 0.005" rpy="0 0 0"/>
+      <origin xyz="0 0 0.03" rpy="0 0 0"/>
       <inertia ixx="1e-6" ixy="0" ixz="0" iyy="1e-6" iyz="0" izz="1e-6" />
     </inertial>
     <collision>
-      <origin xyz="0 0 0.005" rpy="0 0 0"/>
+      <origin xyz="0 0 0.03" rpy="0 0 0"/>
       <geometry>
         <box size="0.01 0.05 0.015"/>
@@ -15,5 +15,5 @@
     </collision>
     <visual>
-      <origin xyz="0 0 0.005" rpy="0 0 0"/>
+      <origin xyz="0 0 0.03" rpy="0 0 0"/>
       <geometry>
         <box size="0.01 0.05 0.015"/>
@@ -23,5 +23,5 @@
   </link>
   <joint name="zed_camera_joint" type="fixed">
-    <origin xyz="0.0 0.0 0.005" rpy="0.0 0.1 2.3" />
+    <origin xyz="0.0 0.0 0.03" rpy="0.0 0.1 2.3" />
     <parent link="drone/base_link"/>
     <child link="zed_camera_link"/>
@@ -34,10 +34,10 @@
     <inertial>
       <mass value="1e-3" />
-      <origin xyz="0 0 0.005" rpy="0 0 0"/>
+      <origin xyz="0 0 0.03" rpy="0 0 0"/>
       <inertia ixx="1e-6" ixy="0" ixz="0" iyy="1e-6" iyz="0" izz="1e-6" />
     </inertial>
   </link>
   <joint name="zed_camera_left_joint" type="fixed">
-    <origin xyz="0 0 0.005" rpy="0 0 0"/>
+    <origin xyz="0 0 0.03" rpy="0 0 0"/>
     <parent link="zed_camera_link"/>
     <child link="camera_link"/>
